File: ECAD/keyboard.kicad_sch (KiCad schematic)
At the start: 9 parts, among them P1 USB_C_Plug_USB2.0, SW91 RotaryEncoder_Switch

Commit message: Updated Schematic
Parts:
- removed ESP1, ESP2: ~, symbol ESP_Custom:AITRIP_ESP32
- added U2: SC1512_13_-A4, SC1512_13_-A4:QFN40P1000X1000X90-81N, symbol SC1512_13_-A4:SC1512_13_-A4
Connections:
- net  Bluetooth: now also U2.27 (GPIO26)
- net 2.4: now also U2.26 (GPIO25)
- net Col0: now also U2.77 (GPIO0)
- net Col1: now also U2.78 (GPIO1)
- net Col2: now also U2.79 (GPIO2)
- net Col3: now also U2.80 (GPIO3)
- net Col4: now also U2.1 (GPIO4)
- net Col5: now also U2.2 (GPIO5)
- net Col6: now also U2.3 (GPIO6)
- net Col7: now also U2.4 (GPIO7)
- net Col8: now also U2.6 (GPIO8)
- net LED D Out: now also U2.49 (GPIO40_ADC0)
- net RotaryA: now also U2.21 (GPIO21)
- net RotaryB: now also U2.20 (GPIO20)
- net RotarySwitch: now also U2.19 (GPIO19)
- net Row0: now also U2.7 (GPIO9)
- net Row1: now also U2.8 (GPIO10)
- net Row2: now also U2.9 (GPIO11)
- net Row3: now also U2.11 (GPIO12)
- net Row4: now also U2.12 (GPIO13)
- net Row5: now also U2.13 (GPIO14)
- net Row6: now also U2.14 (GPIO15)
- net Row7: now also U2.16 (GPIO16)
- net Row8: now also U2.17 (GPIO17)
- net Row9: now also U2.18 (GPIO18)
- net SDA: now also U2.40 (GPIO32)
- net SLC: now also U2.39 (GPIO31)
- net USB D+: now also U2.67 (USB_DP)
- net USB D-: now also U2.66 (USB_DM)
- net Wired: now also U2.25 (GPIO24)
- new net CE: U2.28 (GPIO27)
- new net IUSB1: U2.36 (GPIO28)
- new net IUSB2: U2.37 (GPIO29)
- new net IUSB3: U2.38 (GPIO30)
Other:
- sheet Power ports: added CE, IUSB1, IUSB2, IUSB3; removed Charge%
