File: ECAD/power.kicad_sch (KiCad schematic)
At the start: 1 part

Commit message: Updated Schematic
Parts:
- added C1, C2: 4.7 uF, symbol Device:C
- added C3, C5: 1uF, symbol Device:C
- added C4: 0.01uF, symbol Device:C
- added C6, C7: 10uF, symbol Device:C
- added D211, D212: LED, symbol Device:LED
- added L1: 2.2uH, symbol Device:L
- added Q1: NMOS_Substrate, symbol Simulation_SPICE:NMOS_Substrate
- added R2: R(ISET), symbol Device:R_US
- added U1: BQ24166RGE, Package_DFN_QFN:Texas_RGE0024H_VQFN-24-1EP_4x4mm_P0.5mm_EP2.7x2.7mm, symbol Battery_Management:BQ24166RGE
Connections:
- net USB V BUS: now also C1.1, U1.22 (USB)
- net at BT1.1 (+): now also C3.1, Q1.1 (D), U1.11 (BAT), U1.12 (BAT)
- net GND: now reaches BT1.2 (-)
- net GND: now also C1.2, C2.2, C3.2, C5.2, C6.2, C7.1, Q1.2 (G), R2.2, U1.16 (PGND), U1.17 (PGND), U1.25 (PGND)
- new net: C4.2, L1.1, U1.18 (SW)
- new net: C2.1, U1.23 (PMIDU)
- new net: Q1.4 (Bulk), U1.10 (BGATE)
- new net: R2.1, U1.5 (ISET)
- new net: C4.1, U1.19 (BOOT)
- new net: C5.1, D211.2 (A), D212.2 (A), U1.6 (DRV)
- new net: D211.1 (K), U1.7 (~{PG})
- new net: D212.1 (K), U1.8 (~{CHG})
- new net CE: U1.24 (~{CE})
- new net IUSB1: U1.4 (IUSB1)
- new net IUSB2: U1.3 (IUSB2)
- new net IUSB3: U1.2 (IUSB3)
- new net PNGD: C6.1, C7.2, L1.2, Q1.3 (S), U1.13 (SYS), U1.14 (SYS)
- no-connect marks 0 -> 5
Other:
- moved on the sheet: BT1
